Commit message: .

File: ROS/mybot_description/urdf/mybot.xacro (robot description, xacro)
@@ -9,5 +9,6 @@
   <xacro:include filename="$(find mybot_description)/urdf/macros.xacro" />
 -->
-  <link name='chassis'>
+<!-- CHASSIS -->
+  <link name="chassis">
     <pose>0 0 0.1 0 0 0</pose>
     <inertial>
@@ -32,4 +33,27 @@
     </visual>
   </link>
+<!-- CAMERA -->
+<link name="camera">
+        <collision name="collision_camera">
+                <origin xyz="0 0 0.028575" rpy="0 0 0" />
+                <geometry>
+                         <box size="0.1 0.1 0.1" />
+                </geometry>
+        </collision>
+	<visual name="camera_visual">
+                <origin xyz="0 0 0.028575" rpy="0 0 0" />
+                <geometry>
+                        <box size="0.1 0.1 0.1" />
+                </geometry>
+        </visual>
+        <inertial>
+                <mass value="0.1" />
+                <origin xyz="0 0 0.0001" rpy="0 0 0"/>
+                <inertia ixx="0.0001" ixy="0.0" ixz="0.0"
+                         iyy="0.0001" iyz="0.0"
+                         izz="0.0001" />
+        </inertial>
+</link>
+<!-- WHEEL LINKS -->
   <link name="left_wheel">
     <!--origin xyz="0.1 0.13 0.1" rpy="0 1.5707 1.5707"-->
@@ -128,4 +152,5 @@
     </inertial>
   </link>
+<!-- WHEEL JOINTS -->
   <joint type="continuous" name="left_wheel_hinge">
     <origin xyz="0.1 0.15 0" rpy="0 0 0"/>
@@ -160,3 +185,9 @@
     <joint_properties damping="0.0" friction="1"/>
   </joint>
+<joint name="kinect_joint" type="fixed">
+        <origin xyz="-0.15 0 0.1" rpy="0 0 3.1414" />
+        <child link="camera" />
+        <parent link="chassis" />
+</joint>
+<!-- END -->
 </robot>
